File: nubus-to-ztex/nubus.sch (KiCad schematic (older format))
At the start: 66 parts, among them J4 C96ABC, U1 74LVT125, U2 74LVT125, U3 74LVT125, U4 XC9572XL-VQ64, U5 74LVT245BPW,118, U6 74LVT245BPW,118, U7 74LVT245BPW,118, U8 74LVT245BPW,118

Commit message: forgot to commit last attempt at V1.2
Parts:
- removed C10, C12, C16, C9: 100nF, Capacitor_SMD:C_0603_1608Metric, symbol Device:C
- removed C13: 1uF, Capacitor_SMD:C_0603_1608Metric, symbol Device:C
- removed C15: 10nF, Capacitor_SMD:C_0603_1608Metric, symbol Device:C
- removed D10, D15, D16, D6, D7, D8, D9: YELLOW, LED_SMD:LED_0805_2012Metric, symbol Device:LED_ALT
- removed D4, D5: ORANGE, LED_SMD:LED_0805_2012Metric, symbol Device:LED_ALT
- removed R10, R11, R12, R13, R14, R15, R20, R21, R9: 549, Resistor_SMD:R_0603_1608Metric, symbol Device:R
- removed U4: XC9572XL-VQ64, For_SeeedStudio:TQFP-64_10x10mm_P0.5mm_Xlinx, symbol CPLD_Xilinx:XC9572XL-VQ64
- added C30: 100nF, Capacitor_SMD:C_0603_1608Metric, symbol Device:C
- added U12: 74CB3T1G125DBVR, Package_TO_SOT_SMD:SOT-23-5, symbol 74xGxx:74CB3T1G125
- added U13, U4: SN74CB3T3125PWR, Package_SO:TSSOP-14_4.4x5mm_P0.65mm, symbol ul_SN74CB3T3125PW:SN74CB3T3125PW
- added U14: SN74CB3T3245PWR, For_SeeedStudio:TSSOP-20_4.4x6.5mm_P0.65mm_ForSeeedStudio, symbol SN74CB3T3245PWR:SN74CB3T3245PWR
- C11, C7, C8: value 10nF -> 100nF; MPN CC0603KRX7R8BB103 -> CC0603KRX7R8BB104; Mouser 603-CC603KRX7R8BB103 -> 603-CC603KRX7R8BB104; URL https://lcsc.com/product-detail/Multilayer-Ceramic-Capacito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 -> (none)
Connections:
- net +3V3: now also C30.1, U13.14 (VCC), U14.20 (VCC), U4.14 (VCC)
- net GND: now also C30.2, U12.1 (~OE), U12.3 (GND), U13.1 (*1OE), U13.10 (*3OE), U13.13 (*4OE), U13.4 (*2OE), U13.7 (GND), U14.10 (GND), U14.19 (~OE), U4.1 (*1OE), U4.10 (*3OE), U4.13 (*4OE), U4.4 (*2OE), U4.7 (GND)
- net ~ACK_3V3: now also U4.5 (2A)
- net ~ACK_5V: now also U4.6 (2B)
- net ~ARB0_5V: now also U14.8 (A7)
- net ~ARB1_5V: now also U14.9 (A8)
- net ~ARB2_5V: now also U14.6 (A5)
- net ~ARB3_5V: now also U14.7 (A6)
- net ~CLK2X_3V3: now also U12.4 (B)
- net ~CLK2X_5V: now also U12.2 (A)
- net ~CLK_3V3: now also U4.9 (3A)
- net ~CLK_5V: now also U4.8 (3B)
- net ~ID0_3V3: now also U14.15 (B4)
- net ~ID0_5V: now also U14.5 (A4)
- net ~ID1_3V3: now also U14.16 (B3)
- net ~ID1_5V: now also U14.4 (A3)
- net ~ID2_3V3: now also U14.17 (B2)
- net ~ID2_5V: now also U14.3 (A2)
- net ~ID3_3V3: now also U14.18 (B1)
- net ~ID3_5V: now also U14.2 (A1)
- net ~RESET_3V3: now also U13.12 (4A)
- net ~RESET_5V: now also U13.11 (4B)
- net ~RQST_3V3: now also U4.2 (1A)
- net ~RQST_5V: now also U4.3 (1B)
- net ~START_3V3: now also U4.12 (4A)
- net ~START_5V: now also U4.11 (4B)
- net ~TM0_3V3: now also U13.5 (2A)
- net ~TM0_5V: now also U13.6 (2B)
- net ~TM1_3V3: now also U13.2 (1A)
- net ~TM1_5V: now also U13.3 (1B)
- net ~TM2_3V3: now also U13.9 (3A)
- net ~TM2_5V: now also U13.8 (3B)
- new net VCC: U12.5 (VCC)
- new net ~ARB0_3V3: U14.12 (B7)
- new net ~ARB1_3V3: U14.11 (B8)
- new net ~ARB2_3V3: U14.14 (B5)
- new net ~ARB3_3V3: U14.13 (B6)
Other:
- note added: "For ID, it's likely all Macs are using open/ground,\nso we could pull-up to +3V3 and avoid the level shifter entirely."
- note added: "Slot ID Leds\n(pull-ups are on the 5V side of the shifters)"
- note added: "always enabled"
- note removed: "Internal signal tap leds"
- note removed: "Signals Tap Leds"
- note removed: "Slot ID Leds\n(pull-ups are on the 5V side of the CPLD)"
- moved on the sheet: R5, R6, R7, R8

Commit message: more stuff thinking about V1.2
Other:
- note added: "signals formerly from FPGA to CPLD\nTBC they are no longer needed"
Changed lines of the file:
@@
 Text Notes 6400 13700 0    50   ~ 0
 always enabled
+Wire Notes Line
+	6950 8450 7850 8450
+Wire Notes Line
+	7850 8450 7850 9300
+Wire Notes Line
+	7850 9300 6950 9300
+Wire Notes Line
+	6950 9300 6950 8450
+Text Notes 6750 8450 0    50   ~ 0
+signals formerly from FPGA to CPLD\nTBC they are no longer needed
 $EndSCHEMATC
