File: nubus-to-ztex/nubus.sch (KiCad schematic (older format))
At the start: 54 parts, among them J4 C96ABC, U1 74LVT125, U13 SN74CB3T3245PWR, U14 SN74CB3T3245PWR, U15 SN74CB3T3245PWR, U2 74LVT125, U3 74LVT125, U5 74LVT245BPW,118, U6 74LVT245BPW,118, U7 74LVT245BPW,118, U8 74LVT245BPW,118

Commit message: more update to V1.2 to try to limit cost
Parts:
- D10, D6, D7, D8, D9: value YELLOW -> YELLOW Led
- D11, D12, D13, D14: value GREEN -> GREEN Led
- J4: value C96ABC -> 0850030567 (DIN 41612C 3x32 pins)
- U1, U2, U3: value 74LVT125 -> 74LVT125PW,118
Changed lines of the file:
@@
 P 22250 5750
 F 0 "J4" H 22429 5846 50  0000 L CNN
-F 1 "C96ABC" H 22429 5755 50  0000 L CNN
+F 1 "0850030567 (DIN 41612C 3x32 pins)" H 22429 5755 50  0000 L CNN
 F 2 "For_SeeedStudio:DIN41612_C_3x32_Male_Horizontal_THT" H 22250 5800 50  0001 C CNN
 F 3 " ~" H 22250 5800 50  0001 C CNN
@@
 AR Path="/618F532C/61D85DFA" Ref="D11"  Part="1"
 F 0 "D11" H 16050 7950 50  0000 C CNN
-F 1 "GREEN" H 16100 7700 50  0000 R CNN
+F 1 "GREEN Led" H 16100 7700 50  0000 R CNN
 F 2 "LED_SMD:LED_0805_2012Metric" H 16050 7850 50  0001 C CNN
 F 3 "https://www.lcsc.com/product-detail/Light-Emitting-Diodes-LED_Lite-On-LTST-C170KGKT_C98221.html" H 16050 7850 50  0001 C CNN
@@
 AR Path="/618F532C/61D85E17" Ref="D12"  Part="1"
 F 0 "D12" H 16050 8450 50  0000 C CNN
-F 1 "GREEN" H 16100 8200 50  0000 R CNN
+F 1 "GREEN Led" H 16100 8200 50  0000 R CNN
 F 2 "LED_SMD:LED_0805_2012Metric" H 16050 8350 50  0001 C CNN
 F 3 "https://www.lcsc.com/product-detail/Light-Emitting-Diodes-LED_Lite-On-LTST-C170KGKT_C98221.html" H 16050 8350 50  0001 C CNN
@@
 AR Path="/618F532C/61D85E34" Ref="D13"  Part="1"
 F 0 "D13" H 16050 8950 50  0000 C CNN
-F 1 "GREEN" H 16100 8700 50  0000 R CNN
+F 1 "GREEN Led" H 16100 8700 50  0000 R CNN
 F 2 "LED_SMD:LED_0805_2012Metric" H 16050 8850 50  0001 C CNN
 F 3 "https://www.lcsc.com/product-detail/Light-Emitting-Diodes-LED_Lite-On-LTST-C170KGKT_C98221.html" H 16050 8850 50  0001 C CNN
@@
 AR Path="/618F532C/61D85E51" Ref="D14"  Part="1"
 F 0 "D14" H 16050 9450 50  0000 C CNN
-F 1 "GREEN" H 16100 9200 50  0000 R CNN
+F 1 "GREEN Led" H 16100 9200 50  0000 R CNN
 F 2 "LED_SMD:LED_0805_2012Metric" H 16050 9350 50  0001 C CNN
 F 3 "https://www.lcsc.com/product-detail/Light-Emitting-Diodes-LED_Lite-On-LTST-C170KGKT_C98221.html" H 16050 9350 50  0001 C CNN
@@
 P 4050 5900
 F 0 "U3" H 4050 6217 50  0000 C CNN
-F 1 "74LVT125" H 4050 6126 50  0000 C CNN
+F 1 "74LVT125PW,118" H 4050 6126 50  0000 C CNN
 F 2 "Package_SO:TSSOP-14_4.4x5mm_P0.65mm" H 4050 5900 50  0001 C CNN
 F 3 "http://www.ti.com/lit/gpn/sn74LVT125" H 4050 5900 50  0001 C CNN
@@
 P 4050 6350
 F 0 "U3" H 4050 6667 50  0000 C CNN
-F 1 "74LVT125" H 4050 6576 50  0000 C CNN
+F 1 "74LVT125PW,118" H 4050 6576 50  0000 C CNN
 F 2 "Package_SO:TSSOP-14_4.4x5mm_P0.65mm" H 4050 6350 50  0001 C CNN
 F 3 "http://www.ti.com/lit/gpn/sn74LVT125" H 4050 6350 50  0001 C CNN
@@
 P 4050 6850
 F 0 "U3" H 4050 7167 50  0000 C CNN
-F 1 "74LVT125" H 4050 7076 50  0000 C CNN
+F 1 "74LVT125PW,118" H 4050 7076 50  0000 C CNN
 F 2 "Package_SO:TSSOP-14_4.4x5mm_P0.65mm" H 4050 6850 50  0001 C CNN
 F 3 "http://www.ti.com/lit/gpn/sn74LVT125" H 4050 6850 50  0001 C CNN
@@
 P 4050 7350
 F 0 "U3" H 4050 7667 50  0000 C CNN
-F 1 "74LVT125" H 4050 7576 50  0000 C CNN
+F 1 "74LVT125PW,118" H 4050 7576 50  0000 C CNN
 F 2 "Package_SO:TSSOP-14_4.4x5mm_P0.65mm" H 4050 7350 50  0001 C CNN
 F 3 "http://www.ti.com/lit/gpn/sn74LVT125" H 4050 7350 50  0001 C CNN
@@
 P 5500 6550
 F 0 "U3" H 5730 6596 50  0000 L CNN
-F 1 "74LVT125" H 5730 6505 50  0000 L CNN
+F 1 "74LVT125PW,118" H 5730 6505 50  0000 L CNN
 F 2 "Package_SO:TSSOP-14_4.4x5mm_P0.65mm" H 5500 6550 50  0001 C CNN
 F 3 "http://www.ti.com/lit/gpn/sn74LVT125" H 5500 6550 50  0001 C CNN
@@
 P 3450 2500
 F 0 "U1" H 3450 2817 50  0000 C CNN
-F 1 "74LVT125" H 3450 2726 50  0000 C CNN
+F 1 "74LVT125PW,118" H 3450 2726 50  0000 C CNN
 F 2 "Package_SO:TSSOP-14_4.4x5mm_P0.65mm" H 3450 2500 50  0001 C CNN
 F 3 "http://www.ti.com/lit/gpn/sn74LVT125" H 3450 2500 50  0001 C CNN
@@
 P 3450 2950
 F 0 "U1" H 3450 3267 50  0000 C CNN
-F 1 "74LVT125" H 3450 3176 50  0000 C CNN
+F 1 "74LVT125PW,118" H 3450 3176 50  0000 C CNN
 F 2 "Package_SO:TSSOP-14_4.4x5mm_P0.65mm" H 3450 2950 50  0001 C CNN
 F 3 "http://www.ti.com/lit/gpn/sn74LVT125" H 3450 2950 50  0001 C CNN
@@
 P 3450 3400
 F 0 "U1" H 3450 3717 50  0000 C CNN
-F 1 "74LVT125" H 3450 3626 50  0000 C CNN
+F 1 "74LVT125PW,118" H 3450 3626 50  0000 C CNN
 F 2 "Package_SO:TSSOP-14_4.4x5mm_P0.65mm" H 3450 3400 50  0001 C CNN
 F 3 "http://www.ti.com/lit/gpn/sn74LVT125" H 3450 3400 50  0001 C CNN
@@
 P 3450 3850
 F 0 "U1" H 3450 4167 50  0000 C CNN
-F 1 "74LVT125" H 3450 4076 50  0000 C CNN
+F 1 "74LVT125PW,118" H 3450 4076 50  0000 C CNN
 F 2 "Package_SO:TSSOP-14_4.4x5mm_P0.65mm" H 3450 3850 50  0001 C CNN
 F 3 "http://www.ti.com/lit/gpn/sn74LVT125" H 3450 3850 50  0001 C CNN
@@
 P 5050 3200
 F 0 "U1" H 5280 3246 50  0000 L CNN
-F 1 "74LVT125" H 5280 3155 50  0000 L CNN
+F 1 "74LVT125PW,118" H 5280 3155 50  0000 L CNN
 F 2 "Package_SO:TSSOP-14_4.4x5mm_P0.65mm" H 5050 3200 50  0001 C CNN
 F 3 "http://www.ti.com/lit/gpn/sn74LVT125" H 5050 3200 50  0001 C CNN
@@
 P 3650 10150
 F 0 "U2" H 3650 10467 50  0000 C CNN
-F 1 "74LVT125" H 3650 10376 50  0000 C CNN
+F 1 "74LVT125PW,118" H 3650 10376 50  0000 C CNN
 F 2 "Package_SO:TSSOP-14_4.4x5mm_P0.65mm" H 3650 10150 50  0001 C CNN
 F 3 "http://www.ti.com/lit/gpn/sn74LVT125" H 3650 10150 50  0001 C CNN
@@
 P 3650 11050
 F 0 "U2" H 3650 11367 50  0000 C CNN
-F 1 "74LVT125" H 3650 11276 50  0000 C CNN
+F 1 "74LVT125PW,118" H 3650 11276 50  0000 C CNN
 F 2 "Package_SO:TSSOP-14_4.4x5mm_P0.65mm" H 3650 11050 50  0001 C CNN
 F 3 "http://www.ti.com/lit/gpn/sn74LVT125" H 3650 11050 50  0001 C CNN
@@
 P 3650 11500
 F 0 "U2" H 3650 11817 50  0000 C CNN
-F 1 "74LVT125" H 3650 11726 50  0000 C CNN
+F 1 "74LVT125PW,118" H 3650 11726 50  0000 C CNN
 F 2 "Package_SO:TSSOP-14_4.4x5mm_P0.65mm" H 3650 11500 50  0001 C CNN
 F 3 "http://www.ti.com/lit/gpn/sn74LVT125" H 3650 11500 50  0001 C CNN
@@
 P 5100 10650
 F 0 "U2" H 5330 10696 50  0000 L CNN
-F 1 "74LVT125" H 5330 10605 50  0000 L CNN
+F 1 "74LVT125PW,118" H 5330 10605 50  0000 L CNN
 F 2 "Package_SO:TSSOP-14_4.4x5mm_P0.65mm" H 5100 10650 50  0001 C CNN
 F 3 "http://www.ti.com/lit/gpn/sn74LVT125" H 5100 10650 50  0001 C CNN
@@
 P 3650 10600
 F 0 "U2" H 3650 10917 50  0000 C CNN
-F 1 "74LVT125" H 3650 10826 50  0000 C CNN
+F 1 "74LVT125PW,118" H 3650 10826 50  0000 C CNN
 F 2 "Package_SO:TSSOP-14_4.4x5mm_P0.65mm" H 3650 10600 50  0001 C CNN
 F 3 "http://www.ti.com/lit/gpn/sn74LVT125" H 3650 10600 50  0001 C CNN
@@
 AR Path="/6332A9A8/6332F9B3" Ref="D?"  Part="1"
 F 0 "D6" H 13000 7850 50  0000 C CNN
-F 1 "YELLOW" H 13050 7600 50  0000 R CNN
+F 1 "YELLOW Led" H 13050 7600 50  0000 R CNN
 F 2 "LED_SMD:LED_0805_2012Metric" H 13000 7750 50  0001 C CNN
 F 3 "https://lcsc.com/product-detail/Light-Emitting-Diodes-LED_Lite-On-LTST-C170KSKT_C125091.html" H 13000 7750 50  0001 C CNN
@@
 AR Path="/6332A9A8/63342049" Ref="D?"  Part="1"
 F 0 "D9" H 13000 9100 50  0000 C CNN
-F 1 "YELLOW" H 13050 8850 50  0000 R CNN
+F 1 "YELLOW Led" H 13050 8850 50  0000 R CNN
 F 2 "LED_SMD:LED_0805_2012Metric" H 13000 9000 50  0001 C CNN
 F 3 "https://lcsc.com/product-detail/Light-Emitting-Diodes-LED_Lite-On-LTST-C170KSKT_C125091.html" H 13000 9000 50  0001 C CNN
@@
 AR Path="/6332A9A8/63343356" Ref="D?"  Part="1"
 F 0 "D10" H 13000 9550 50  0000 C CNN
-F 1 "YELLOW" H 13050 9300 50  0000 R CNN
+F 1 "YELLOW Led" H 13050 9300 50  0000 R CNN
 F 2 "LED_SMD:LED_0805_2012Metric" H 13000 9450 50  0001 C CNN
 F 3 "https://lcsc.com/product-detail/Light-Emitting-Diodes-LED_Lite-On-LTST-C170KSKT_C125091.html" H 13000 9450 50  0001 C CNN
@@
 AR Path="/6332A9A8/6334A05C" Ref="D?"  Part="1"
 F 0 "D7" H 13000 8250 50  0000 C CNN
-F 1 "YELLOW" H 13050 8000 50  0000 R CNN
+F 1 "YELLOW Led" H 13050 8000 50  0000 R CNN
 F 2 "LED_SMD:LED_0805_2012Metric" H 13000 8150 50  0001 C CNN
 F 3 "https://lcsc.com/product-detail/Light-Emitting-Diodes-LED_Lite-On-LTST-C170KSKT_C125091.html" H 13000 8150 50  0001 C CNN
@@
 AR Path="/6332A9A8/63352DC7" Ref="D?"  Part="1"
 F 0 "D8" H 13000 8650 50  0000 C CNN
-F 1 "YELLOW" H 13050 8400 50  0000 R CNN
+F 1 "YELLOW Led" H 13050 8400 50  0000 R CNN
 F 2 "LED_SMD:LED_0805_2012Metric" H 13000 8550 50  0001 C CNN
 F 3 "https://lcsc.com/product-detail/Light-Emitting-Diodes-LED_Lite-On-LTST-C170KSKT_C125091.html" H 13000 8550 50  0001 C CNN
